File: PCB/Night-Gogle MKI/Night-Gogle.kicad_pcb (KiCad board)
At the start: 2 copper layers, 83 x 43.5 mm, 27 parts, among them J1 Conn_01x08_Pin, SW1 SW_Push, U1 IRL540N

Commit message: pcb update
Parts:
- removed GND2: ~, N-G_board:Pad-3.5mm
- added GND: ~, N-G_board:Pad-3.5mm, F.Cu at (93.0, 69.6)
- added IR-LED: ~, N-G_board:Pad-3.5mm, F.Cu at (86.5, 69.6)
- IR: renamed from IR-Led2; moved to B.Cu
- R1: footprint Resistor_THT:R_Axial_DIN0411_L9.9mm_D3.6mm_P12.70mm_Horizontal -> Resistor_SMD:R_0805_2012Metric_Pad1.20x1.40mm_HandSolder
- R2, R3, R4, R5: footprint Resistor_THT:R_Axial_DIN0411_L9.9mm_D3.6mm_P12.70mm_Horizontal -> Resistor_SMD:R_1206_3216Metric_Pad1.30x1.75mm_HandSolder
- VIN: renamed from VIN2; moved to B.Cu
- moved R1 88.4 mm to (85.0, 64.3), turned to 90 degrees
- moved U1 80.0 mm to (89.8, 57.6), turned to 90 degrees
- moved R4 67.5 mm to (107.2, 85.2), turned to -90 degrees
- moved R3 64.3 mm to (124.4, 83.9)
- moved D5 61.1 mm to (112.9, 85.9), turned to 180 degrees
- moved D3 56.2 mm to (125.2, 78.2), turned to -90 degrees
- moved D6 55.4 mm to (119.7, 85.9), turned to 180 degrees
- moved D4 47.7 mm to (125.2, 71.4), turned to -90 degrees
- moved R2 34.0 mm to (105.9, 67.9), turned to 180 degrees
- moved IR 21.6 mm to (117.7, 62.2), turned to 180 degrees
- moved R5 18.9 mm to (123.2, 66.7), turned to 90 degrees
- moved VIN 16.2 mm to (112.9, 62.2), turned to 180 degrees
- moved D7 5.84 mm to (117.4, 65.9)
- moved D8 5.84 mm to (110.7, 65.9)
- moved D2 4.11 mm to (105.2, 73.7)
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- renumbered GND1 to GND, IR-LED1 to IR-LED, VIN1 to VIN
Routing:
- net +5V: track 32.9 -> 120.0 mm, vias 2 -> 3
- net IR-In: track 0.00 -> 80.5 mm
- net Button1: track 13.8 -> 23.9 mm, vias 1 -> 2
- net IR-Led: track 22.4 -> 27.5 mm
- net Net-(D5-K): track 0.00 -> 4.24 mm
- net Net-(D3-K): track 0.00 -> 4.24 mm
- net Net-(D7-K): track 0.00 -> 4.21 mm
- net Net-(D1-A): track 0.00 -> 4.20 mm
- net Net-(D3-A): track 0.00 -> 4.17 mm
- net Net-(D2-A): track 0.00 -> 4.16 mm
- net Net-(D7-A): track 0.00 -> 4.16 mm
- net Net-(D5-A): track 0.00 -> 4.16 mm
- net Net-(R1-Pad2): track 0.00 -> 2.48 mm
- net GND: vias 0 -> 2
Other:
- board size 83 x 43.5 mm -> 81.2 x 45.2 mm

Commit message: gg
Parts:
- added R6: 10K, Resistor_SMD:R_0805_2012Metric_Pad1.20x1.40mm_HandSolder, F.Cu at (89.8, 65.0)
- R2, R3, R4, R5: value 100R -> 160R
- moved D1 10.9 mm to (116.0, 78.6)
- moved VIN 10.9 mm to (123.7, 60.3)
- moved D2 10.9 mm to (116.0, 71.8)
- moved D5 10.9 mm to (123.7, 84.1)
- moved D8 10.9 mm to (121.5, 64.1)
- moved R2 10.9 mm to (116.7, 66.1)
- moved R4 10.9 mm to (118.0, 83.3)
- moved D3 10.9 mm to (135.9, 76.3)
- moved D4 10.9 mm to (135.9, 69.5)
- moved D6 10.9 mm to (130.5, 84.1)
- moved D7 10.9 mm to (128.2, 64.1)
- moved IR-Led 10.9 mm to (128.4, 60.3)
- moved R3 10.9 mm to (135.2, 82.1)
- moved R5 10.9 mm to (133.9, 64.8)
- renumbered IR to IR-Led
Connections:
- IR-Led pad 1: IR-Led -> IR-In
Routing:
- net GND: track 0.00 -> 1.95 mm
- net Net-(R1-Pad2): track 2.48 -> 4.43 mm
Other:
- board size 81.2 x 45.2 mm -> 91.9 x 43.5 mm

Commit message: Big Update
Parts:
- J1: value Conn_01x08_Pin -> Conn_01x06_Pin; footprint Connector_JST:JST_SH_BM08B-SRSS-TB_1x08-1MP_P1.00mm_Vertical -> Connector_JST:JST_SH_SM06B-SRSS-TB_1x06-1MP_P1.00mm_Horizontal
- moved D1 12.2 mm to (106.2, 86.0)
- moved D2 12.2 mm to (106.2, 79.2)
- moved D5 12.2 mm to (114.0, 91.5)
- moved D8 12.2 mm to (111.8, 71.5)
- moved R2 12.2 mm to (107.0, 73.5)
- moved R4 12.2 mm to (108.2, 90.8)
- moved VIN2 12.2 mm to (114.0, 67.8)
- moved D3 12.2 mm to (126.2, 83.7)
- moved D4 12.2 mm to (126.2, 77.0)
- moved D6 12.2 mm to (120.8, 91.5)
- moved D7 12.2 mm to (118.5, 71.5)
- moved IR-Led2 12.2 mm to (118.8, 67.8)
- moved R3 12.2 mm to (125.5, 89.5)
- moved R5 12.2 mm to (124.2, 72.2)
- moved J1 1.00 mm to (65.5, 53.0)
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- renumbered GND to GND1, GND to GND2, IR-LED to IR-LED1, IR-LED to IR-LED3, IR-Led to IR-Led2, VIN to VIN1, VIN to VIN2
Connections:
- J1 pad 1: BLK -> RST
- J1 pad 2: CS -> DC
- J1 pad 3: DC -> CS
- J1 pad 4: RST -> SCLK
- J1 pad 6: SCLK -> GND
- MCU1 pad P$16: +3.3V -> unconnected-(MCU1-3V3-PadP$16)
- MCU1 pad P$3: RST -> MOSI
- MCU1 pad P$4: MOSI -> SCLK
- MCU1 pad P$5: DC -> CS
- MCU1 pad P$6: SCLK -> DC
- MCU1 pad P$7: CS -> RST
- MCU1 pad P$8: BLK -> unconnected-(MCU1-IO4-PadP$8)
Routing:
- net BLK: track 25.6 -> 0.00 mm, vias 1 -> 0
- net +3.3V: track 15.7 -> 0.00 mm, vias 1 -> 0
- net RST: track 15.9 -> 27.7 mm
- net DC: track 20.5 -> 26.1 mm
- net MOSI: track 17.8 -> 15.1 mm
- net CS: track 23.6 -> 21.2 mm
- net SCLK: track 18.4 -> 19.6 mm, vias 0 -> 1
- net Button1: track 23.9 -> 22.9 mm
- net +5V: track 120.0 -> 119.9 mm, vias 3 -> 1
- net GND: vias 2 -> 0
Other:
- board size 91.9 x 43.5 mm -> 82.2 x 50.8 mm
